File: schemat_KiCad/PŁYTKA PRZEDNIA/płytka_przednia.kicad_pcb (KiCad board)
At the start: 2 copper layers, 124.6 x 39.1 mm, 25 parts, among them T1 KTIR0711S, T2 KTIR0711S, T3 KTIR0711S, T4 KTIR0711S, T5 KTIR0711S, T6 KTIR0711S, T7 KTIR0711S, T8 KTIR0711S

Commit message: tył do druku
Parts:
- removed R11, R21, R31, R41, R51, R61, R71, R81: 200, Resistors_SMD:R_0805_HandSoldering
- removed R12: 10K, Resistors_SMD:R_0805_HandSoldering
- removed R22, R32, R42, R52, R62, R72, R82: 10k, Resistors_SMD:R_0805_HandSoldering
- removed T1, T2, T3, T4, T5, T6, T7, T8: KTIR0711S, warsztaty:KTIR0711S
- removed WYJŚCIE_PLYTKA_TYLNIA1: PIN10, warsztatymisc:fpc_10_pin
Routing:
- net GND: track 174.0 -> 0.00 mm, vias 3 -> 0
- net VCC: track 156.6 -> 0.00 mm, vias 1 -> 0
- net /T8: track 60.0 -> 0.00 mm, vias 1 -> 0
- net /T1: track 48.9 -> 0.00 mm, vias 1 -> 0
- net /T7: track 45.6 -> 0.00 mm, vias 1 -> 0
- net (no net): track 42.6 -> 0.00 mm, vias 2 -> 0
- net /T2: track 40.4 -> 0.00 mm, vias 1 -> 0
- net /T6: track 33.8 -> 0.00 mm, vias 2 -> 0
- net /T3: track 29.9 -> 0.00 mm, vias 1 -> 0
- net /T4: track 17.6 -> 0.00 mm, vias 1 -> 0
- net /T5: track 17.4 -> 0.00 mm, vias 2 -> 0
- net Net-(R11-Pad2): track 8.44 -> 0.00 mm
- net Net-(R21-Pad2): track 4.68 -> 0.00 mm
- net Net-(R71-Pad2): track 3.88 -> 0.00 mm
- net Net-(R81-Pad2): track 3.57 -> 0.00 mm
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- removed copper zone on B.Cu, net GND
- removed copper zone on F.Cu, net GND
Other:
- board outline removed
- board text removed: "BEBO"
