File: schemat_KiCad/EENKODERY/enkodery.kicad_pcb (KiCad board)
At the start: 2 copper layers, 25.5 x 18 mm, 4 parts, among them J1 CONN_01X08

Commit message: poprawiony echo/trig
Routing:
- net /3V3: track 47.8 -> 45.7 mm
Other:
- outline, holes or cut-outs redrawn
Changed lines of the file:
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@@
     (thickness 1.6)
     (drawings 6)
-    (tracks 77)
+    (tracks 83)
     (zones 0)
     (modules 4)
@@
   )
   (setup
-    (last_trace_width 0.25)
+    (last_trace_width 0.4)
     (user_trace_width 0.4)
     (trace_clearance 0.2)
@@
     (trace_min 0.2)
     (segment_width 0.2)
-    (edge_width 0.15)
+    (edge_width 0.2)
     (via_size 0.6)
     (via_drill 0.4)
@@
   (gr_line (start 175 78) (end 149.5 78) (angle 90) (layer Edge.Cuts) (width 0.15))
   (gr_line (start 175 96) (end 149.5 96) (angle 90) (layer Edge.Cuts) (width 0.15))
-  (gr_circle (center 151.5 94.1) (end 152.5 94.6) (layer F.Fab) (width 0.2))
-  (gr_circle (center 151.5 80.1) (end 152 81.1) (layer F.Fab) (width 0.2))
+  (gr_circle (center 151.5 94.1) (end 152.5 94.6) (layer Edge.Cuts) (width 0.2))
+  (gr_circle (center 151.5 80.1) (end 152 81.1) (layer Edge.Cuts) (width 0.2))
   (gr_line (start 175 78) (end 175 96) (angle 90) (layer Edge.Cuts) (width 0.15))
+  (segment (start 154.955 84.455) (end 154.935 84.455) (width 0.4) (layer F.Cu) (net 7))
+  (segment (start 154.935 84.455) (end 154.04 85.35) (width 0.4) (layer F.Cu) (net 7))
+  (segment (start 154.35 85.35) (end 154.39 85.35) (width 0.4) (layer F.Cu) (net 7))
+  (segment (start 167.5011 80.0036) (end 159.4064 80.0036) (width 0.4) (layer F.Cu) (net 7))
+  (segment (start 158.535 80.875) (end 159.4064 80.0036) (width 0.4) (layer F.Cu) (net 7))
+  (segment (start 158.535 80.875) (end 154.955 84.455) (width 0.4) (layer F.Cu) (net 7))
+  (segment (start 154.955 85.955) (end 154.93 85.93) (width 0.4) (layer F.Cu) (net 7))
   (segment (start 158.25 87.25) (end 158.25 87.3) (width 0.4) (layer F.Cu) (net 7))
   (segment (start 158.25 87.3) (end 157.8964 87.6536) (width 0.4) (layer F.Cu) (net 7))
@@
   (segment (start 164.9 80.9) (end 160.9 80.9) (width 0.4) (layer F.Cu) (net 7))
   (segment (start 166.0036 82.0036) (end 164.9 80.9) (width 0.4) (layer F.Cu) (net 7))
-  (segment (start 167.5011 80.0036) (end 155.6964 80.0036) (width 0.4) (layer F.Cu) (net 7))
-  (segment (start 154.6 81.1) (end 154.6 85.6) (width 0.4) (layer F.Cu) (net 7))
-  (segment (start 155.6964 80.0036) (end 154.6 81.1) (width 0.4) (layer F.Cu) (net 7))
-  (segment (start 152.75 85.35) (end 154.35 85.35) (width 0.4) (layer F.Cu) (net 7))
+  (segment (start 152.75 85.35) (end 154.04 85.35) (width 0.4) (layer F.Cu) (net 7))
+  (segment (start 154.04 85.35) (end 154.35 85.35) (width 0.4) (layer F.Cu) (net 7))
   (segment (start 154.35 85.35) (end 154.6 85.6) (width 0.4) (layer F.Cu) (net 7))
-  (segment (start 154.6 85.6) (end 156.0036 87.0036) (width 0.4) (layer F.Cu) (net 7))
+  (segment (start 154.6 85.6) (end 154.93 85.93) (width 0.4) (layer F.Cu) (net 7))
+  (segment (start 154.93 85.93) (end 156.0036 87.0036) (width 0.4) (layer F.Cu) (net 7))
   (segment (start 156.0036 87.0036) (end 156.9761 87.0036) (width 0.4) (layer F.Cu) (net 7))
   (segment (start 156.9761 87.6536) (end 157.8964 87.6536) (width 0.4) (layer F.Cu) (net 7))
