File: schemat_KiCad/EENKODERY/enkodery.sch (KiCad schematic (older format))
At the start: 4 parts, among them J1 CONN_01X08

Commit message: archiwum ze złego projektu + drukowanie
Parts:
- J1: footprint Pin_Headers:Pin_Header_Angled_1x08_Pitch2.00mm -> Pin_Headers:Pin_Header_Straight_1x08_Pitch2.00mm
Changed lines of the file:
@@
 F 0 "J1" H 6850 5150 50  0000 C CNN
 F 1 "CONN_01X08" V 6950 4700 50  0000 C CNN
-F 2 "Pin_Headers:Pin_Header_Angled_1x08_Pitch2.00mm" H 6850 4700 50  0001 C CNN
+F 2 "Pin_Headers:Pin_Header_Straight_1x08_Pitch2.00mm" H 6850 4700 50  0001 C CNN
 F 3 "" H 6850 4700 50  0001 C CNN
 	1    6850 4700
