File: schemat_KiCad/PŁYTKA TYLNIA/plytka_tylnia.kicad_pcb (KiCad board)
At the start: 2 copper layers, 135 x 101 mm, 62 parts, among them J1 CONN_01X04, J2 PIN8, J3 PIN8, P1 USB_OTG

Commit message: skompletowane czesci, wybrane rezystory, kondensator przy wejsciu
Parts:
- added C18: 100nF, Capacitors_SMD:C_0805_HandSoldering, F.Cu at (125.2, 58.7)
- C10: value 1uF -> 10uF
- C11: value 10uF -> 100nF
- C13: value 0.1uF -> 100nF
- R10: value R -> 220R
- R11: value R -> 43k
- R12: value R -> 13k
- R13: value R -> 56k
- R14: value R -> 51k
- R15: value R -> 33k
- R2: moved to B.Cu
- R4: value R -> 160k
- R5: value R -> 20k
- R9: value R -> 10k
- moved R2 55.0 mm to (155.5, 55.4), turned to 90 degrees
- moved P1 1.89 mm to (93.1, 59.8), turned to 225 degrees
- moved REF** 0.07 mm to (87.4, 117.5)
Routing:
- net VCC: track 448.2 -> 427.1 mm
- net /SPI1_MISO: track 137.5 -> 142.3 mm
- net /SWCLK: track 88.0 -> 91.3 mm
- net /SWDIO: track 102.9 -> 105.9 mm
- net /RESET: track 130.4 -> 133.0 mm, vias 4 -> 3
- net /5V: track 347.0 -> 345.5 mm
- net GND: track 766.2 -> 765.4 mm, vias 6 -> 7
- net /SPI1_MOSI: track 142.3 -> 141.8 mm

Commit message: archiwum ze złego projektu + drukowanie
Parts:
- moved P1 3.66 mm to (95.7, 57.2)
- moved J2 0.62 mm to (110.0, 124.6)
- moved J3 0.55 mm to (165.0, 110.5)
Routing:
- net GND: track 765.4 -> 770.5 mm
- net Net-(MOSTEK1-Pad1): track 104.6 -> 108.5 mm
- net VCC: track 427.1 -> 423.8 mm
- net /SWDIO: track 105.9 -> 102.5 mm
- net /SWCLK: track 91.3 -> 88.6 mm
- net /SPI1_MISO: track 142.3 -> 144.0 mm
- net /5V: track 345.5 -> 347.0 mm
- net /SPI1_SS2: track 103.5 -> 102.4 mm
- net /SPI1_SS1: track 148.3 -> 147.4 mm
- net /RESET: track 133.0 -> 133.8 mm
- net /SPI1_MOSI: track 141.8 -> 141.0 mm, vias 3 -> 2
