File: schemat_KiCad/PŁYTKA(bez turbiny)/plytka_tylnia.sch (KiCad schematic (older format))
At the start: 80 parts, among them J1 CONN_01X04, J2 CONN_01X04, J3 CONN_01X04, J4 CONN_01X04, J5 CONN_01X04, J6 CONN_01X04, J7 PIN10, J8 CONN_01X04, J9 CONN_01X04, P1 USB_OTG, T1 KTIR0711S, T2 KTIR0711S, T3 KTIR0711S, T4 KTIR0711S, T5 KTIR0711S, T6 KTIR0711S, T7 KTIR0711S, T8 KTIR0711S, U1 AS5048A, U2 AS5048A

Commit message: poprawiona, odchudzona, zaokraglona
Parts:
- added BATERIA?: LI-POL, misc:zl_zasilania, symbol CONN_01X02
- added Bezpiecznik?: Fuse ??, Fuse_Holders_and_Fuses:Fuse_SMD1206_HandSoldering, symbol Fuse
- added C? (x2): 10uF, Capacitors_Tantalum_SMD:CP_Tantalum_Case-A_EIA-3216-18_Hand, symbol CP
- added C? (x2): 100nF, symbol C
- added C? (x2): 10uF, symbol CP
- added J?: CONN_02X20, symbol CONN_02X20
- added J? (x2): CONN_01X20, symbol CONN_01X20
- added Q? (x2): BSS138, TO_SOT_Packages_SMD:SOT-23, symbol 2N7002
- added R?: 1k, Resistors_SMD:R_0805_HandSoldering, symbol R
- added R? (x2): 10k, symbol R
- added STABILIZATOR?: LM1117, warsztaty:LM1117_TO-252, symbol LM1117
- added TRANSISTOR?: BUZ11, misc:SOT23-3, symbol BUZ11
- added Włącznik?: switch, misc:tact_switch_smd, symbol SPST
Connections:
- net BATERIA: now also Bezpiecznik?.1, C?.1, R?.1, STABILIZATOR?.1 (VI)
- new net: BATERIA?.1 (P1), TRANSISTOR?.3 (D)
- new net: BATERIA?.2 (P2), Włącznik?.1
- new net: R?.2, TRANSISTOR?.1 (G)
- new net: Bezpiecznik?.2, Włącznik?.2
- new net: Q?.2 (S), R?.2
- new net: Q?.3 (D), Q?.3 (D)
- new net: Q?.2 (S), R?.1
- new net GND3: C?.2, C?.2, C?.2, C?.2, C?.2, C?.2, J?.10 (P10), J?.12 (P12), J?.14 (P14), J?.16 (P16), J?.18 (P18), J?.2 (P2), J?.20 (P20), J?.22 (P22), J?.24 (P24), J?.26 (P26), J?.28 (P28), J?.30 (P30), J?.32 (P32), J?.34 (P34), J?.36 (P36), J?.38 (P38), J?.4 (P4), J?.40 (P40), J?.6 (P6), J?.8 (P8), STABILIZATOR?.3 (GND), TRANSISTOR?.2 (S)
- new net PWM5V: J?.1 (P1), J?.10 (P10), J?.11 (P11), J?.12 (P12), J?.13 (P13), J?.14 (P14), J?.15 (P15), J?.16 (P16), J?.17 (P17), J?.18 (P18), J?.19 (P19), J?.2 (P2), J?.20 (P20), J?.3 (P3), J?.4 (P4), J?.5 (P5), J?.6 (P6), J?.7 (P7), J?.8 (P8), J?.9 (P9)
- new net VCC3: C?.1, C?.1, C?.1, J?.1 (P1), J?.11 (P11), J?.13 (P13), J?.15 (P15), J?.17 (P17), J?.19 (P19), J?.21 (P21), J?.23 (P23), J?.25 (P25), J?.27 (P27), J?.29 (P29), J?.3 (P3), J?.31 (P31), J?.33 (P33), J?.35 (P35), J?.37 (P37), J?.39 (P39), J?.5 (P5), J?.7 (P7), J?.9 (P9), Q?.1 (G), R?.1, STABILIZATOR?.2 (VO)
- new net VCC5: C?.1, C?.1, Q?.1 (G), R?.2
Other:
- moved on the sheet: C16, J7, R1, R11, R12, R13, R14, R15, R16, R17, R18, R19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
